Commit message: Add realtip on urdf

File: openteach/robot/assets/robot.urdf (robot description, URDF)
Before this commit: robot onshape, 17 links, 16 joints
Links:
- added link realtip, mass 0.1; collision sphere radius=0.005; visual sphere radius=0.005
- added link realtip_2, mass 0.1; collision sphere radius=0.005; visual sphere radius=0.005
- added link realtip_3, mass 0.1; collision sphere radius=0.005; visual sphere radius=0.005
- added link realtip_4, mass 0.1; collision sphere radius=0.005; visual sphere radius=0.005
- link dip: geometry collision mesh filename=package://leap_hand/meshes//dip.stl; visual mesh filename=package://leap_hand/meshes//dip.stl
- link dip_2: geometry collision mesh filename=package://leap_hand/meshes//dip.stl; visual mesh filename=package://leap_hand/meshes//dip.stl
- link dip_3: geometry collision mesh filename=package://leap_hand/meshes//dip.stl; visual mesh filename=package://leap_hand/meshes//dip.stl
- link fingertip: geometry collision mesh filename=package://leap_hand/meshes//fingertip.stl; visual mesh filename=package://leap_hand/meshes//fingertip.stl
- link fingertip_2: geometry collision mesh filename=package://leap_hand/meshes//fingertip.stl; visual mesh filename=package://leap_hand/meshes//fingertip.stl
- link fingertip_3: geometry collision mesh filename=package://leap_hand/meshes//fingertip.stl; visual mesh filename=package://leap_hand/meshes//fingertip.stl
- link mcp_joint: geometry collision mesh filename=package://leap_hand/meshes//mcp_joint.stl; visual mesh filename=package://leap_hand/meshes//mcp_joint.stl
- link mcp_joint_2: geometry collision mesh filename=package://leap_hand/meshes//mcp_joint.stl; visual mesh filename=package://leap_hand/meshes//mcp_joint.stl
- link mcp_joint_3: geometry collision mesh filename=package://leap_hand/meshes//mcp_joint.stl; visual mesh filename=package://leap_hand/meshes//mcp_joint.stl
- link palm_lower: geometry collision mesh filename=package://leap_hand/meshes//palm_lower.stl; visual mesh filename=package://leap_hand/meshes//palm_lower.stl
- link pip: geometry collision mesh filename=package://leap_hand/meshes//pip.stl; visual mesh filename=package://leap_hand/meshes//pip.stl
- link pip_2: geometry collision mesh filename=package://leap_hand/meshes//pip.stl; visual mesh filename=package://leap_hand/meshes//pip.stl
- link pip_3: geometry collision mesh filename=package://leap_hand/meshes//pip.stl; visual mesh filename=package://leap_hand/meshes//pip.stl
- link pip_4: geometry collision mesh filename=package://leap_hand/meshes//pip.stl; visual mesh filename=package://leap_hand/meshes//pip.stl
- link thumb_dip: geometry collision mesh filename=package://leap_hand/meshes//thumb_dip.stl; visual mesh filename=package://leap_hand/meshes//thumb_dip.stl
- link thumb_fingertip: geometry collision mesh filename=package://leap_hand/meshes//thumb_fingertip.stl; visual mesh filename=package://leap_hand/meshes//thumb_fingertip.stl
- link thumb_pip: geometry collision mesh filename=package://leap_hand/meshes//thumb_pip.stl; visual mesh filename=package://leap_hand/meshes//thumb_pip.stl
Joints:
- added joint 16: type fixed, parent fingertip, child realtip, origin xyz=-0.01 -0.05 0.015 rpy=4.5935029425113685044e-17 -2.8730071914463794583e-16 4.4395481053923607589e-32, axis 0 0 -1, limit lower=-0.366 upper=2.042 effort=0.95 velocity=8.48
- added joint 17: type fixed, parent fingertip_2, child realtip_2, origin xyz=-0.01 -0.05 0.015 rpy=4.5935029425113685044e-17 -2.8730071914463794583e-16 4.4395481053923607589e-32, axis 0 0 -1, limit lower=-0.366 upper=2.042 effort=0.95 velocity=8.48
- added joint 18: type fixed, parent fingertip_3, child realtip_3, origin xyz=-0.01 -0.05 0.015 rpy=4.5935029425113685044e-17 -2.8730071914463794583e-16 4.4395481053923607589e-32, axis 0 0 -1, limit lower=-0.366 upper=2.042 effort=0.95 velocity=8.48
- added joint 19: type fixed, parent thumb_fingertip, child realtip_4, origin xyz=-0.01 -0.06 -0.015 rpy=4.5935029425113685044e-17 -2.8730071914463794583e-16 4.4395481053923607589e-32, axis 0 0 -1, limit lower=-0.366 upper=2.042 effort=0.95 velocity=8.48
- joint 0: limit lower=-1.047 upper=1.047 effort=0.95 velocity=8.48 -> lower=-1.047 upper=0.1 effort=0.95 velocity=8.48
- joint 14: limit lower=-1.2 upper=1.90 effort=0.95 velocity=8.48 -> lower=-1.20 upper=1.90 effort=0.95 velocity=8.48
- joint 4: limit lower=-1.047 upper=1.047 effort=0.95 velocity=8.48 -> lower=-0.3 upper=0.3 effort=0.95 velocity=8.48
- joint 8: limit lower=-1.047 upper=1.047 effort=0.95 velocity=8.48 -> lower=-0.1 upper=1.047 effort=0.95 velocity=8.48
